Commit message: working version

File: urdf/fra2mo.xacro (robot description, xacro)
@@ -3,5 +3,5 @@
   <xacro:include filename="$(find rl_fratomo_description)/urdf/fratomo_base_macro.xacro" />
   <xacro:include filename="$(find rl_fratomo_description)/urdf/lidar_gazebo_macro.xacro" />
-  <!--<xacro:include filename="$(find rl_fratomo_description)/urdf/d435_gazebo_macro.xacro" />-->
+  <!-- <xacro:include filename="$(find rl_fratomo_description)/urdf/d435_gazebo_macro.xacro" /> --> <!-- Uncomment if you want to add also a D435 camera -->
   <xacro:property name="LIDAR" value="True"/>
   <xacro:property name="DEPTH" value="True"/>
@@ -12,4 +12,5 @@
     <xacro:lidar_gazebo_sensor parent="lidar_link" />
   </xacro:if>
+  <!-- Uncomment if you want to add also a D435 camera -->
   <!-- RGBD Sensor
   <xacro:if value="${DEPTH}" >

File: urdf/fra2mo_base_macro.xacro (robot description, xacro)
@@ -85,6 +85,7 @@
       </inertial>
     </link>
-    <link name="d435_link">
-    </link>
+    <!-- Uncomment if you want to add also a D435 camera -->
+    <!-- <link name="d435_link">
+    </link> -->
     <link name="lidar_link">
     </link>

Commit message: name conflicts solved

File: urdf/fra2mo.xacro (robot description, xacro)
@@ -1,11 +1,11 @@
 <?xml version="1.0"?>
-<robot name="fratomo" xmlns:xacro="http://ros.org/wiki/xacro">
-  <xacro:include filename="$(find rl_fratomo_description)/urdf/fratomo_base_macro.xacro" />
-  <xacro:include filename="$(find rl_fratomo_description)/urdf/lidar_gazebo_macro.xacro" />
-  <!-- <xacro:include filename="$(find rl_fratomo_description)/urdf/d435_gazebo_macro.xacro" /> --> <!-- Uncomment if you want to add also a D435 camera -->
+<robot name="fra2mo" xmlns:xacro="http://ros.org/wiki/xacro">
+  <xacro:include filename="$(find rl_fra2mo_description)/urdf/fra2mo_base_macro.xacro" />
+  <xacro:include filename="$(find rl_fra2mo_description)/urdf/lidar_gazebo_macro.xacro" />
+  <xacro:include filename="$(find rl_fra2mo_description)/urdf/d435_gazebo_macro.xacro" /> <!--Uncomment if you want to add also a D435 camera-->
   <xacro:property name="LIDAR" value="True"/>
   <xacro:property name="DEPTH" value="True"/>
   <!-- Diff Drive Robot Base  -->
-  <xacro:fratomo_base />
+  <xacro:fra2mo_base />
   <!-- LIDAR Sensor -->
   <xacro:if value="${LIDAR}" >
@@ -13,7 +13,7 @@
   </xacro:if>
   <!-- Uncomment if you want to add also a D435 camera -->
-  <!-- RGBD Sensor
+  <!-- RGBD Sensor -->
   <xacro:if value="${DEPTH}" >
     <xacro:d435_gazebo_sensor parent="d435_link" />
-  </xacro:if>   -->
+  </xacro:if>
 </robot>

File: urdf/fra2mo_base_macro.xacro (robot description, xacro)
@@ -1,5 +1,5 @@
 <?xml version="1.0"?>
-<robot name="fratomo_base_macro" xmlns:xacro="http://www.ros.org/wiki/xacro">
-  <xacro:include filename="$(find rl_fratomo_description)/urdf/utility_macro.xacro" />
+<robot name="fra2mo_base_macro" xmlns:xacro="http://www.ros.org/wiki/xacro">
+  <xacro:include filename="$(find rl_fra2mo_description)/urdf/utility_macro.xacro" />
   <!-- Base properties -->
 	<xacro:property name="base_height" value="0.180" />
@@ -10,5 +10,5 @@
   <xacro:property name="wheel_axle" value="0.130" />
   <!-- WHOLE BASE MACRO-->
-  <xacro:macro name="fratomo_base" > <!--fb : front, back ; lr: left, right -->
+  <xacro:macro name="fra2mo_base" > <!--fb : front, back ; lr: left, right -->
       <!--Actual body/chassis of the robot-->
     <link name="base_footprint">
@@ -23,5 +23,5 @@
       <visual>
         <geometry>
-          <mesh filename="package://rl_fratomo_description/meshes/rl_fratomo_body.stl" scale="0.001 0.001 0.001 "/>
+          <mesh filename="package://rl_fra2mo_description/meshes/rl_fra2mo_body.stl" scale="0.001 0.001 0.001 "/>
         </geometry>
         <material name="White"/>
@@ -44,5 +44,5 @@
       <visual>
         <geometry>
-          <mesh filename="package://rl_fratomo_description/meshes/rl_fratomo_wheel.stl" scale="0.001 0.001 0.001 "/>
+          <mesh filename="package://rl_fra2mo_description/meshes/rl_fra2mo_wheel.stl" scale="0.001 0.001 0.001 "/>
         </geometry>
         <material name="Black"/>
@@ -51,5 +51,5 @@
       <collision>
         <geometry>
-          <mesh filename="package://rl_fratomo_description/meshes/rl_fratomo_wheel.stl" scale="0.001 0.001 0.001 "/>
+          <mesh filename="package://rl_fra2mo_description/meshes/rl_fra2mo_wheel.stl" scale="0.001 0.001 0.001 "/>
         </geometry>
         <origin rpy="0 0 0" xyz="0 0 0"/>
@@ -66,5 +66,5 @@
       <visual>
         <geometry>
-          <mesh filename="package://rl_fratomo_description/meshes/rl_fratomo_wheel.stl" scale="0.001 0.001 0.001 "/>
+          <mesh filename="package://rl_fra2mo_description/meshes/rl_fra2mo_wheel.stl" scale="0.001 0.001 0.001 "/>
         </geometry>
         <material name="Black"/>
@@ -73,5 +73,5 @@
       <collision>
         <geometry>
-          <mesh filename="package://rl_fratomo_description/meshes/rl_fratomo_wheel.stl" scale="0.001 0.001 0.001 "/>
+          <mesh filename="package://rl_fra2mo_description/meshes/rl_fra2mo_wheel.stl" scale="0.001 0.001 0.001 "/>
         </geometry>
         <origin rpy="0 0 0" xyz="0 0 0"/>
@@ -86,6 +86,6 @@
     </link>
     <!-- Uncomment if you want to add also a D435 camera -->
-    <!-- <link name="d435_link">
-    </link> -->
+    <link name="d435_link">
+    </link>
     <link name="lidar_link">
     </link>

File: urdf/lidar_gazebo_macro.xacro (robot description, xacro)
@@ -12,5 +12,5 @@
       <visual>
         <geometry>
-          <mesh filename="package://rl_fratomo_description/meshes/lidar.stl" scale="0.001 0.001 0.001 "/>
+          <mesh filename="package://rl_fra2mo_description/meshes/lidar.stl" scale="0.001 0.001 0.001 "/>
         </geometry>
         <material name="White"/>
