Commit message: first commit, it is possible to visualize on rviz and gazebo

File: urdf/d435_gazebo_macro.xacro (robot description, xacro)
@@ -1,19 +1,16 @@
 <?xml version="1.0"?>
-<robot name="lidar_gazebo_macro" xmlns:xacro="http://www.ros.org/wiki/xacro">
-  <!--xacro:include filename="$(find rl_fratomo_description)/urdf/utility_macro.xacro" /-->
+<robot name="d435_gazebo_macro" xmlns:xacro="http://ros.org/wiki/xacro">
   <xacro:include filename="$(find realsense2_description)/urdf/_d435.urdf.xacro" />
-  <xacro:macro name="d435_gazebo_sensor" params="parent" >
+  <xacro:macro name="d435_gazebo_sensor" params="parent">
     <xacro:sensor_d435 parent="${parent}" use_nominal_extrinsics="true" add_plug="false" use_mesh="true">
-      <origin xyz="0 0 0" rpy="0 0 0"/>
+      <origin xyz="0 0 0" rpy="0 0 0" />
     </xacro:sensor_d435>
     <gazebo reference="${parent}">
-      <sensor type="depth" name="$depth_camera">
+      <sensor type="depth_camera" name="depth_camera">
         <always_on>true</always_on>
         <update_rate>30.0</update_rate>
         <camera>
-          <!--horizontal_fov>2</horizontal_fov-->
           <horizontal_fov>1.3962634</horizontal_fov>
           <image>
-            <!--format>L8</format-->
             <format>BGR8</format>
             <width>640</width>
@@ -25,21 +22,14 @@
           </clip>
         </camera>
-        <plugin name="depth_camera_plugin" filename="libgazebo_ros_openni_kinect.so">
-          <alwaysOn>true</alwaysOn>
-          <baseline>0.11</baseline>
-          <updateRate>30.0</updateRate>
-          <cameraName>depth_camera</cameraName>
-          <imageTopicName>depth_camera/image_raw</imageTopicName>
-          <cameraInfoTopicName>depth_camera/camera_info</cameraInfoTopicName>
-          <depthImageTopicName>depth/disparity</depthImageTopicName>
-          <depthImageCameraInfoTopicName>depth/camera_info</depthImageCameraInfoTopicName>
-          <pointCloudTopicName>depth/points</pointCloudTopicName>
-          <frameName>camera_depth_optical_frame</frameName>
-          <pointCloudCutoff>0.5</pointCloudCutoff>
-          <distortionK1>0.0</distortionK1>
-          <distortionK2>0.0</distortionK2>
-          <distortionK3>0.0</distortionK3>
-          <distortionT1>0.0</distortionT1>
-          <distortionT2>0.0</distortionT2>
+        <plugin name="GazeboRosDepthCamera" filename="libgazebo_ros_depth_camera.so">
+          <ros>
+            <namespace>/</namespace>
+            <remapping>~/depth/image_raw:=/depth_camera/image_raw</remapping>
+            <remapping>~/depth/camera_info:=/depth_camera/camera_info</remapping>
+            <remapping>~/points:=/depth/points</remapping>
+          </ros>
+          <update_rate>30.0</update_rate>
+          <camera_name>depth_camera</camera_name>
+          <frame_name>camera_depth_optical_frame</frame_name>
         </plugin>
       </sensor>

File: urdf/fra2mo_base_macro.xacro (robot description, xacro)
@@ -1,161 +1,140 @@
 <?xml version="1.0"?>
-<robot name="fra2mo_base_macro" xmlns:xacro="http://www.ros.org/wiki/xacro">
+<robot  xmlns:xacro="http://www.ros.org/wiki/xacro">
   <xacro:include filename="$(find rl_fra2mo_description)/urdf/utility_macro.xacro" />
-  <!-- Base properties -->
-	<xacro:property name="base_height" value="0.180" />
-  <xacro:property name="base_radius" value="0.11" />
-  <xacro:property name="base_mass" value="5" />
-  <xacro:property name="wheel_mass" value="2.5" />
-  <xacro:property name="wheel_radius" value="0.035" />
-  <xacro:property name="wheel_axle" value="0.130" />
   <!-- WHOLE BASE MACRO-->
   <xacro:macro name="fra2mo_base" > <!--fb : front, back ; lr: left, right -->
-      <!--Actual body/chassis of the robot-->
+    <!-- Base properties -->
+    <xacro:property name="base_height" value="0.180" />
+    <xacro:property name="base_radius" value="0.11" />
+    <xacro:property name="base_mass" value="5" />
+    <xacro:property name="wheel_mass" value="2.5" />
+    <xacro:property name="wheel_radius" value="0.035" />
+    <xacro:property name="wheel_axle" value="0.130" />
+    <!-- Actual body/chassis of the robot -->
     <link name="base_footprint">
     </link>
     <link name="base_link">
+      <!-- Inertial properties -->
       <inertial>
-          <inertia ixx="1.0" ixy="0.0" ixz="0.0" iyy="1.0" iyz="0.0" izz="1.0"/>
+        <origin xyz="0 0 0" />
         <mass value="${base_mass}" />
-        <origin xyz="0 0 0" />
-        <cylinder_inertia  m="${base_mass}" r="${base_radius}" h="${base_height}" />
+        <xacro:cylinder_inertia m="${base_mass}" r="${base_radius}" h="${base_height}" />
       </inertial>
+      <!-- Visual representation -->
       <visual>
         <geometry>
-          <mesh filename="package://rl_fra2mo_description/meshes/rl_fra2mo_body.stl" scale="0.001 0.001 0.001 "/>
+          <mesh filename="file://$(find rl_fra2mo_description)/meshes/rl_fra2mo_body.stl" scale="0.001 0.001 0.001" />
         </geometry>
-        <material name="White"/>
-        <origin rpy="0 0 0" xyz="0 0 0"/>
+        <material name="White" />
+        <origin xyz="0 0 0" rpy="0 0 0" />
+      </visual>
+      <!-- Collision properties -->
+      <collision>
+        <geometry>
+          <cylinder length="${base_height}" radius="${base_radius}" />
+        </geometry>
+        <origin xyz="0 0.0 ${(base_height/2.0)-0.05}" rpy="0 0 0" />
+      </collision>
+      <collision>
+        <geometry>
+          <sphere radius="0.019" />
+        </geometry>
+        <origin xyz="-0.0825 0.0 -0.04" rpy="0 0 0" />
+      </collision>
+    </link>
+    <!-- Left Wheel -->
+    <link name="left_wheel_link">
+      <visual>
+        <geometry>
+          <mesh filename="file://$(find rl_fra2mo_description)/meshes/rl_fra2mo_wheel.stl" scale="0.001 0.001 0.001" />
+        </geometry>
+        <material name="Black" />
+        <origin xyz="0 0 0" rpy="0 0 0" />
       </visual>
       <collision>
         <geometry>
-          <cylinder length="${base_height}" radius="${base_radius}"/>
+          <mesh filename="file://$(find rl_fra2mo_description)/meshes/rl_fra2mo_wheel.stl" scale="0.001 0.001 0.001" />
         </geometry>
-        <origin rpy="0 0 0" xyz="0 0.0 ${(base_height/2.0)-0.05}"/>
+        <origin xyz="0 0 0" rpy="0 0 0" />
       </collision>
-      <collision>
-        <geometry>
-          <sphere radius="0.019"/>
-        </geometry>
-        <origin rpy="0 0 0" xyz="-0.0825 0.0 -0.04"/>
-      </collision>
+      <inertial>
+        <origin xyz="0 0 0" />
+        <mass value="${wheel_mass}" />
+        <inertia ixx="0.001" ixy="0.0" ixz="0.0" iyy="0.001" iyz="0.0" izz="0.001" />
+      </inertial>
     </link>
-    <link name="left_wheel_link">
+    <!-- Right Wheel -->
+    <link name="right_wheel_link">
       <visual>
         <geometry>
-          <mesh filename="package://rl_fra2mo_description/meshes/rl_fra2mo_wheel.stl" scale="0.001 0.001 0.001 "/>
+          <mesh filename="file://$(find rl_fra2mo_description)/meshes/rl_fra2mo_wheel.stl" scale="0.001 0.001 0.001" />
         </geometry>
         <material name="Black"/>
-        <origin rpy="0 0 0" xyz="0 0 0"/>
+        <origin xyz="0 0 0" rpy="0 0 0" />
       </visual>
       <collision>
         <geometry>
-          <mesh filename="package://rl_fra2mo_description/meshes/rl_fra2mo_wheel.stl" scale="0.001 0.001 0.001 "/>
+          <mesh filename="file://$(find rl_fra2mo_description)/meshes/rl_fra2mo_wheel.stl" scale="0.001 0.001 0.001" />
         </geometry>
-        <origin rpy="0 0 0" xyz="0 0 0"/>
+        <origin xyz="0 0 0" rpy="0 0 0" />
       </collision>
       <inertial>
+        <origin xyz="0 0 0" />
         <mass value="${wheel_mass}" />
-        <origin xyz="0 0 0" />
-        <inertia ixx="0.001" ixy="0.0" ixz="0.0"
-               iyy="0.001" iyz="0.0"
-               izz="0.001" />
+        <inertia ixx="0.001" ixy="0.0" ixz="0.0" iyy="0.001" iyz="0.0" izz="0.001" />
       </inertial>
     </link>
-    <link name="right_wheel_link">
-      <visual>
-        <geometry>
-          <mesh filename="package://rl_fra2mo_description/meshes/rl_fra2mo_wheel.stl" scale="0.001 0.001 0.001 "/>
-        </geometry>
-        <material name="Black"/>
-        <origin rpy="0 0 0" xyz="0 0 0"/>
-      </visual>
-      <collision>
-        <geometry>
-          <mesh filename="package://rl_fra2mo_description/meshes/rl_fra2mo_wheel.stl" scale="0.001 0.001 0.001 "/>
-        </geometry>
-        <origin rpy="0 0 0" xyz="0 0 0"/>
-      </collision>
-      <inertial>
-        <mass value="${wheel_mass}" />
-        <origin xyz="0 0 0" />
-        <inertia ixx="0.001" ixy="0.0" ixz="0.0"
-               iyy="0.001" iyz="0.0"
-               izz="0.001" />
-      </inertial>
-    </link>
-    <!-- Uncomment if you want to add also a D435 camera -->
-    <link name="d435_link">
-    </link>
-    <link name="lidar_link">
-    </link>
+    <!-- Additional Links -->
+    <link name="d435_link" />
+    <link name="lidar_link" />
+    <!-- Joints -->
     <joint name="base_footprint_joint" type="fixed">
-      <parent link="base_footprint"/>
-      <child link="base_link"/>
-      <origin rpy="0 0 0" xyz="0.0 0.0 0.059"/>
+      <parent link="base_footprint" />
+      <child link="base_link" />
+      <origin xyz="0.0 0.0 0.059" rpy="0 0 0" />
     </joint>
     <joint name="left_wheel_joint" type="continuous">
-      <parent link="base_link"/>
-      <child link="left_wheel_link"/>
-      <origin rpy="0 0 0" xyz="0.04025 0.062 -0.024"/>
-      <axis xyz="0 1 0" rpy="0 0 0" />
-      <limit effort="100" velocity="100"/>
-      <joint_properties damping="0.5" friction="0.01"/>
+      <parent link="base_link" />
+      <child link="left_wheel_link" />
+      <origin xyz="0.04025 0.062 -0.024" rpy="0 0 0" />
+      <axis xyz="0 1 0" />
+      <limit effort="100" velocity="100" />
+      <dynamics damping="0.5" friction="0.01" />
     </joint>
     <joint name="right_wheel_joint" type="continuous">
-      <parent link="base_link"/>
-      <child link="right_wheel_link"/>
-      <origin rpy="0 0 ${-M_PI}" xyz="0.04025 -0.062 -0.024"/>
-      <axis xyz="0 -1 0" rpy="0 0 0" />
-      <limit effort="100" velocity="100"/>
-      <joint_properties damping="0.5" friction="0.01"/>
+      <parent link="base_link" />
+      <child link="right_wheel_link" />
+      <origin xyz="0.04025 -0.062 -0.024" rpy="0 0 ${-M_PI}" />
+      <axis xyz="0 -1 0" />
+      <limit effort="100" velocity="100" />
+      <dynamics damping="0.5" friction="0.01" />
     </joint>
     <joint name="d435_joint" type="fixed">
-      <parent link="base_link"/>
-      <child link="d435_link"/>
-      <origin rpy="0 0 0" xyz="0.090925 0.0 0.06670"/>
+      <parent link="base_link" />
+      <child link="d435_link" />
+      <origin xyz="0.090925 0.0 0.06670" rpy="0 0 0" />
     </joint>
-     <joint name="lidar_joint" type="fixed">
-      <parent link="base_link"/>
-      <child link="lidar_link"/>
-      <origin rpy="0 0 0" xyz="0.0 0.0 0.125"/>
+    <joint name="lidar_joint" type="fixed">
+      <parent link="base_link" />
+      <child link="lidar_link" />
+      <origin xyz="0.0 0.0 0.125" rpy="0 0 0" />
     </joint>
-    <!--gazebo reference="base_link">
-      <mu1 value="0.0"/>
-      <mu2 value="0.0"/>
-      <kp  value="1000000.0" />
-      <kd  value="1.0" />
-      <fdir1 value="1 0 0"/>
-      <material>Gazebo/White</material>
-      <turnGravityOff>false</turnGravityOff>
-    </gazebo-->
-     <gazebo reference="base_link">
+    <!-- Gazebo Material Assignments
+    <gazebo reference="base_link">
       <material>Gazebo/White</material>
     </gazebo>
     <gazebo reference="left_wheel_link">
-      <mu1 value="1.0"/>
-      <mu2 value="1.0"/>
-      <kp  value="1000000.0" />
-      <kd  value="1.0" />
-      <fdir1 value="1 0 0"/>
       <material>Gazebo/Black</material>
-      <turnGravityOff>false</turnGravityOff>
     </gazebo>
-     <gazebo reference="right_wheel_link">
-      <mu1 value="1.0"/>
-      <mu2 value="1.0"/>
-      <kp  value="1000000.0" />
-      <kd  value="1.0" />
-      <fdir1 value="1 0 0"/>
+    <gazebo reference="right_wheel_link">
       <material>Gazebo/Black</material>
-      <turnGravityOff>false</turnGravityOff>
-    </gazebo>
-    <!-- Transmission is important to link the joints and the controller -->
+    </gazebo>-->
+    <!-- Transmissions
     <transmission name="left_wheel_joint_trans">
       <type>transmission_interface/SimpleTransmission</type>
       <joint name="left_wheel_joint" />
       <actuator name="left_wheel_joint_motor">
+        <mechanicalReduction>1</mechanicalReduction>
         <hardwareInterface>EffortJointInterface</hardwareInterface>
-        <mechanicalReduction>1</mechanicalReduction>
       </actuator>
     </transmission>
@@ -164,32 +143,29 @@
       <joint name="right_wheel_joint" />
       <actuator name="right_wheel_joint_motor">
+        <mechanicalReduction>1</mechanicalReduction>
         <hardwareInterface>EffortJointInterface</hardwareInterface>
-        <mechanicalReduction>1</mechanicalReduction>
       </actuator>
-    </transmission>
-     <!-- Differential drive controller  -->
-  <gazebo>
-    <plugin name="differential_drive_controller" filename="libgazebo_ros_diff_drive.so">
-      <legacyMode>true</legacyMode>
-      <rosDebugLevel>Debug</rosDebugLevel>
-      <publishWheelTF>false</publishWheelTF>
-      <robotNamespace>/</robotNamespace>
-      <publishTf>1</publishTf>
-      <publishWheelJointState>true</publishWheelJointState>
-      <alwaysOn>true</alwaysOn>
-      <updateRate>100.0</updateRate>
-      <leftJoint>left_wheel_joint</leftJoint>
-      <rightJoint>right_wheel_joint</rightJoint>
-      <wheelSeparation>${wheel_axle}</wheelSeparation>
-      <wheelDiameter>${2*wheel_radius}</wheelDiameter>
-      <broadcastTF>0</broadcastTF>
-      <wheelTorque>30</wheelTorque>
-      <wheelAcceleration>1.8</wheelAcceleration>
-      <commandTopic>cmd_vel</commandTopic>
-      <odometryFrame>odom</odometryFrame>
-      <odometryTopic>odom</odometryTopic>
-      <robotBaseFrame>base_footprint</robotBaseFrame>
-    </plugin>
-  </gazebo>
-   </xacro:macro>
+    </transmission>-->
+    <!-- Plugin for differential drive control in Gazebo
+    <gazebo>
+      <plugin name="gazebo_ros_diff_drive" filename="libgazebo_ros_diff_drive.so" >
+        <ros>
+          <namespace>/</namespace>
+          <remapping>cmd_vel:=/cmd_vel</remapping>
+        </ros>
+        <update_rate>100.0</update_rate>
+        <left_joint>left_wheel_joint</left_joint>
+        <right_joint>right_wheel_joint</right_joint>
+        <wheel_separation>${wheel_axle}</wheel_separation>
+        <wheel_diameter>${2*wheel_radius}</wheel_diameter>
+        <max_wheel_torque>30</max_wheel_torque>
+        <max_wheel_acceleration>1.8</max_wheel_acceleration>
+        <odom_frame>odom</odom_frame>
+        <robot_base_frame>base_footprint</robot_base_frame>
+        <cmd_vel_topic>cmd_vel</cmd_vel_topic>
+        <odometry_topic>odom</odometry_topic>
+        <publish_joint_states>true</publish_joint_states>
+      </plugin>
+    </gazebo>-->
+  </xacro:macro>
 </robot>

File: urdf/lidar_gazebo_macro.xacro (robot description, xacro)
@@ -1,65 +1,62 @@
 <?xml version="1.0"?>
-<robot name="lidar_gazebo_macro" xmlns:xacro="http://www.ros.org/wiki/xacro">
-  <!--xacro:include filename="$(find rl_fratomo_description)/urdf/utility_macro.xacro" /-->
-  <xacro:macro name="lidar_gazebo_sensor" params="parent" >
+<robot name="lidar_gazebo_macro" xmlns:xacro="http://ros.org/wiki/xacro">
+  <xacro:include filename="$(find rl_fra2mo_description)/urdf/utility_macro.xacro" />
+  <xacro:macro name="lidar_gazebo_sensor" params="parent">
     <link name="laser_frame">
       <inertial>
-          <inertia ixx="1.0" ixy="0.0" ixz="0.0" iyy="1.0" iyz="0.0" izz="1.0"/>
+        <origin xyz="0 0 0" />
         <mass value="0.1" />
-        <origin xyz="0 0 0" />
-        <cylinder_inertia  m="0.1" r="0.037" h="0.04" />
+        <xacro:cylinder_inertia m="0.1" r="0.037" h="0.04" />
       </inertial>
       <visual>
+        <origin rpy="0 0 ${-M_PI_2}" xyz="0.0 0.0 -0.031" />
         <geometry>
-          <mesh filename="package://rl_fra2mo_description/meshes/lidar.stl" scale="0.001 0.001 0.001 "/>
+          <mesh filename="package://rl_fra2mo_description/meshes/lidar.stl" scale="0.001 0.001 0.001" />
         </geometry>
-        <material name="White"/>
-        <origin rpy="0 0 ${-M_PI_2}" xyz="0.0 0.0 -0.031"/>
+        <material name="White" />
       </visual>
       <collision>
-        <origin xyz="0 0 0" rpy="0 0 0 " />
+        <origin xyz="0.0 0.0 -0.031" rpy="0 0 0" />
         <geometry>
           <cylinder length="0.04" radius="0.037" />
         </geometry>
-        <origin rpy="0 0 0" xyz="0.0 0.0 -0.031"/>
       </collision>
     </link>
     <joint name="laser_joint" type="fixed">
-      <parent link="${parent}"/>
-      <child link="laser_frame"/>
-      <origin rpy="0 0 0" xyz="0.0 0.0 0.031"/>
+      <parent link="${parent}" />
+      <child link="laser_frame" />
+      <origin rpy="0 0 0" xyz="0.0 0.0 0.031" />
     </joint>
     <gazebo reference="laser_frame">
-      <sensor type="ray" name="head_hokuyo_sensor">
+      <sensor type="gpu_ray" name="head_hokuyo_sensor">
         <pose>0 0 0 0 0 0</pose>
         <visualize>false</visualize>
         <update_rate>40</update_rate>
-        <ray>
-            <scan>
-              <horizontal>
-                <samples>720</samples>
-                <resolution>1</resolution>
-                <min_angle>-${M_PI} </min_angle>
-                <max_angle>${M_PI} </max_angle>
-              </horizontal>
-            </scan>
-            <range>
-              <min>0.8</min>
-              <max>30.0</max>
-              <resolution>0.01</resolution>
-            </range>
-            <noise>
-              <type>gaussian</type>
-              <!-- Noise parameters based on published spec for Hokuyo laser
-                    achieving "+-30mm" accuracy at range < 10m.  A mean of 0.0m and
-                    stddev of 0.01m will put 99.7% of samples within 0.03m of the true
-                    reading. -->
-              <mean>0.0</mean>
-              <stddev>0.01</stddev>
-            </noise>
-        </ray>
-        <plugin name="gazebo_ros_head_hokuyo_controller" filename="libgazebo_ros_laser.so">
-            <topicName>/laser/scan</topicName>
-            <frameName>laser_frame</frameName>
+        <gpu_ray>
+          <scan>
+            <horizontal>
+              <samples>720</samples>
+              <resolution>1</resolution>
+              <min_angle>${-M_PI}</min_angle>
+              <max_angle>${M_PI}</max_angle>
+            </horizontal>
+          </scan>
+          <range>
+            <min>0.8</min>
+            <max>30.0</max>
+            <resolution>0.01</resolution>
+          </range>
+          <noise>
+            <type>gaussian</type>
+            <mean>0.0</mean>
+            <stddev>0.01</stddev>
+          </noise>
+        </gpu_ray>
+        <plugin name="GazeboRosRaySensor" filename="libgazebo_ros_ray_sensor.so">
+          <ros>
+            <namespace>/</namespace>
+            <remapping>~/LaserScan:=/laser/scan</remapping>
+          </ros>
+          <frameName>laser_frame</frameName>
         </plugin>
       </sensor>

File: urdf/utility_macro.xacro (robot description, xacro)
@@ -1,25 +1,25 @@
 <?xml version="1.0"?>
-<robot name="utility_macro" xmlns:xacro="http://www.ros.org/wiki/xacro">
-  <!--All units in m-kg-s-radians unit system -->
+<robot xmlns:xacro="http://www.ros.org/wiki/xacro">
+  <!-- Tutte le unità nel sistema m-kg-s-radiani -->
   <xacro:property name="M_PI" value="3.1415926535897931" />
   <xacro:property name="M_PI_2" value="1.570796327" />
   <xacro:property name="DEG_TO_RAD" value="0.017453293" />
-	<!--Material Definition-->
-	<material name="Black">
-	  <color rgba="0.0 0.0 0.0 1.0"/>
-	</material>
+  <!-- Definizione dei Materiali -->
+  <material name="Black">
+    <color rgba="0.0 0.0 0.0 1.0" />
+  </material>
   <material name="Red">
-  	<color rgba="0.8 0.0 0.0 1.0"/>
+    <color rgba="0.8 0.0 0.0 1.0" />
   </material>
   <material name="White">
-    <color rgba="1.0 1.0 1.0 1.0"/>
+    <color rgba="1.0 1.0 1.0 1.0" />
   </material>
   <material name="Blue">
-    <color rgba="0.0 0.0 0.8 1.0"/>
+    <color rgba="0.0 0.0 0.8 1.0" />
   </material>
   <xacro:macro name="cylinder_inertia" params="m r h">
-    <inertia  ixx="${m*(3*r*r+h*h)/12}" ixy = "0" ixz = "0"
-              iyy="${m*(3*r*r+h*h)/12}" iyz = "0"
-              izz="${m*r*r/2}" />
+    <inertia ixx="${m*(3*r*r+h*h)/12}" ixy="0" ixz="0"
+             iyy="${m*(3*r*r+h*h)/12}" iyz="0"
+             izz="${(m*r*r)/2}" />
   </xacro:macro>
 </robot>
