Commit message: correcting typo

File: urdf/fra2mo.urdf.xacro (robot description, xacro)
@@ -4,12 +4,12 @@
   <!--<xacro:include filename="$(find rl_fra2mo_description)/urdf/lidar_gazebo_macro.xacro"/> -->
   <!-- <xacro:include filename="$(find rl_fra2mo_description)/urdf/d435_gazebo_macro.xacro" />  -->
-  <!--xacro:property name="LIDAR" value="False"/>
-  <xacro:property name="DEPTH" value="True"/>-->
+  <xacro:property name="LIDAR" value="False"/>
+  <!--<xacro:property name="DEPTH" value="True"/>-->
   <!-- Diff Drive Robot Base -->
   <xacro:fra2mo_base/>
-  <!-- LIDAR Sensor
+  <!-- LIDAR Sensor-->
   <xacro:if value="${LIDAR}">
     <xacro:lidar_gazebo_sensor parent="lidar_link"/>
-  </xacro:if>-->
+  </xacro:if>
   <!-- RGBD Sensor (D435 Camera) -->
   <!--

Commit message: io speriamo che me la cavo

File: urdf/fra2mo.urdf.xacro (robot description, xacro)
@@ -2,7 +2,7 @@
 <robot xmlns:xacro="http://www.ros.org/wiki/xacro" name="fra2mo" >
   <xacro:include filename="$(find rl_fra2mo_description)/urdf/fra2mo_base_macro.xacro"/>
-  <!--<xacro:include filename="$(find rl_fra2mo_description)/urdf/lidar_gazebo_macro.xacro"/> -->
+  <xacro:include filename="$(find rl_fra2mo_description)/urdf/lidar_gazebo_macro.xacro"/>
   <!-- <xacro:include filename="$(find rl_fra2mo_description)/urdf/d435_gazebo_macro.xacro" />  -->
-  <xacro:property name="LIDAR" value="False"/>
+  <xacro:property name="LIDAR" value="True"/>
   <!--<xacro:property name="DEPTH" value="True"/>-->
   <!-- Diff Drive Robot Base -->

File: urdf/fra2mo_base_macro.xacro (robot description, xacro)
@@ -130,5 +130,5 @@
       <material>Gazebo/Black</material>
     </gazebo>-->
-    <!-- Transmissions
+    <!-- Transmissions -->
     <transmission name="left_wheel_joint_trans">
       <type>transmission_interface/SimpleTransmission</type>
@@ -146,26 +146,33 @@
         <hardwareInterface>EffortJointInterface</hardwareInterface>
       </actuator>
-    </transmission>-->
-    <!-- Plugin for differential drive control in Gazebo
+    </transmission>
+    <!-- Plugin for differential drive control in Gazebo-->
     <gazebo>
-      <plugin name="gazebo_ros_diff_drive" filename="libgazebo_ros_diff_drive.so" >
-        <ros>
-          <namespace>/</namespace>
-          <remapping>cmd_vel:=/cmd_vel</remapping>
-        </ros>
-        <update_rate>100.0</update_rate>
-        <left_joint>left_wheel_joint</left_joint>
-        <right_joint>right_wheel_joint</right_joint>
-        <wheel_separation>${wheel_axle}</wheel_separation>
-        <wheel_diameter>${2*wheel_radius}</wheel_diameter>
-        <max_wheel_torque>30</max_wheel_torque>
-        <max_wheel_acceleration>1.8</max_wheel_acceleration>
-        <odom_frame>odom</odom_frame>
-        <robot_base_frame>base_footprint</robot_base_frame>
-        <cmd_vel_topic>cmd_vel</cmd_vel_topic>
-        <odometry_topic>odom</odometry_topic>
-        <publish_joint_states>true</publish_joint_states>
+      <plugin name="ignition::gazebo::systems::DiffDrive" filename="libignition-gazebo-diff-drive-system.so">
+      <left_joint>left_wheel_joint</left_joint>
+      <right_joint>right_wheel_joint</right_joint>
+      <wheel_separation>${wheel_axle}</wheel_separation>
+      <wheel_radius>${wheel_radius}</wheel_radius>
+      <max_wheel_torque>30</max_wheel_torque>
+      <max_wheel_acceleration>1.8</max_wheel_acceleration>
+      <odom_publish_frequency>1</odom_publish_frequency>
+      <!--<ros>
+        <namespace>/fra2mo</namespace>
+        <remapping>cmd_vel:=/cmd_vel</remapping>
+      </ros>
+      <update_rate>100.0</update_rate>
+      <left_joint>left_wheel_joint</left_joint>
+      <right_joint>right_wheel_joint</right_joint>
+      <wheel_separation>${wheel_axle}</wheel_separation>
+      <wheel_radius>${wheel_radius}</wheel_radius>
+      <max_wheel_torque>30</max_wheel_torque>
+      <max_wheel_acceleration>1.8</max_wheel_acceleration>
+      <robot_base_frame>base_footprint</robot_base_frame>
+      <robot_base_frame>base_footprint</robot_base_frame>
+      <cmd_vel_topic>cmd_vel</cmd_vel_topic>
+      <odometry_topic>odom</odometry_topic>
+      <publish_joint_states>true</publish_joint_states>-->
       </plugin>
-    </gazebo>-->
+    </gazebo>
   </xacro:macro>
 </robot>

File: urdf/lidar_gazebo_macro.xacro (robot description, xacro)
@@ -1,5 +1,5 @@
 <?xml version="1.0"?>
-<robot name="lidar_gazebo_macro" xmlns:xacro="http://ros.org/wiki/xacro">
-  <xacro:include filename="$(find rl_fra2mo_description)/urdf/utility_macro.xacro" />
+<robot xmlns:xacro="http://www.ros.org/wiki/xacro" name="lidar_gazebo_macro" >
+  <!--<xacro:include filename="$(find rl_fra2mo_description)/urdf/utility_macro.xacro" />-->
   <xacro:macro name="lidar_gazebo_sensor" params="parent">
     <link name="laser_frame">
@@ -12,5 +12,5 @@
         <origin rpy="0 0 ${-M_PI_2}" xyz="0.0 0.0 -0.031" />
         <geometry>
-          <mesh filename="package://rl_fra2mo_description/meshes/lidar.stl" scale="0.001 0.001 0.001" />
+          <mesh filename="file://$(find rl_fra2mo_description)/meshes/lidar.stl" scale="0.001 0.001 0.001" />
         </geometry>
         <material name="White" />
@@ -22,4 +22,26 @@
         </geometry>
       </collision>
+      <gazebo>
+      <sensor type="gpu_lidar" name="gpu_lidar">
+        <update_rate>40</update_rate>
+        <ray>
+          <scan>
+            <horizontal>
+              <samples>720</samples>
+              <resolution>1</resolution>
+              <min_angle>-3.14</min_angle>
+              <max_angle>3.14</max_angle>
+            </horizontal>
+          </scan>
+          <range>
+            <min>0.1</min>
+            <max>10.0</max>
+            <resolution>0.01</resolution>
+          </range>
+        </ray>
+        <always_on>1</always_on>
+        <visualize>true</visualize>
+      </sensor>
+      </gazebo>
     </link>
     <joint name="laser_joint" type="fixed">
@@ -28,38 +50,4 @@
       <origin rpy="0 0 0" xyz="0.0 0.0 0.031" />
     </joint>
-    <gazebo reference="laser_frame">
-      <sensor type="gpu_ray" name="head_hokuyo_sensor">
-        <pose>0 0 0 0 0 0</pose>
-        <visualize>false</visualize>
-        <update_rate>40</update_rate>
-        <gpu_ray>
-          <scan>
-            <horizontal>
-              <samples>720</samples>
-              <resolution>1</resolution>
-              <min_angle>${-M_PI}</min_angle>
-              <max_angle>${M_PI}</max_angle>
-            </horizontal>
-          </scan>
-          <range>
-            <min>0.8</min>
-            <max>30.0</max>
-            <resolution>0.01</resolution>
-          </range>
-          <noise>
-            <type>gaussian</type>
-            <mean>0.0</mean>
-            <stddev>0.01</stddev>
-          </noise>
-        </gpu_ray>
-        <plugin name="GazeboRosRaySensor" filename="libgazebo_ros_ray_sensor.so">
-          <ros>
-            <namespace>/</namespace>
-            <remapping>~/LaserScan:=/laser/scan</remapping>
-          </ros>
-          <frameName>laser_frame</frameName>
-        </plugin>
-      </sensor>
-    </gazebo>
   </xacro:macro>
 </robot>
