Commit message: added leonardo drone contest world for testing

File: urdf/fra2mo_base_macro.xacro (robot description, xacro)
@@ -26,5 +26,5 @@
           <mesh filename="file://$(find rl_fra2mo_description)/meshes/rl_fra2mo_body.stl" scale="0.001 0.001 0.001" />
         </geometry>
-        <material name="White" />
+        <material name="Blue" />
         <origin xyz="0 0 0" rpy="0 0 0" />
       </visual>
@@ -122,5 +122,5 @@
     <!-- Gazebo Material Assignments
     <gazebo reference="base_link">
-      <material>Gazebo/White</material>
+      <material>Gazebo/Blue</material>
     </gazebo>
     <gazebo reference="left_wheel_link">

Commit message: lidar

File: urdf/fra2mo_base_macro.xacro (robot description, xacro)
@@ -86,5 +86,6 @@
     </link>
     <!-- Additional Links -->
-    <link name="d435_link" />
+    <link name="d435_link">
+    </link>
     <link name="lidar_link" />
     <!-- Joints -->
@@ -150,11 +151,12 @@
     <gazebo>
       <plugin name="ignition::gazebo::systems::DiffDrive" filename="libignition-gazebo-diff-drive-system.so">
-      <left_joint>left_wheel_joint</left_joint>
-      <right_joint>right_wheel_joint</right_joint>
-      <wheel_separation>${wheel_axle}</wheel_separation>
-      <wheel_radius>${wheel_radius}</wheel_radius>
-      <max_wheel_torque>30</max_wheel_torque>
-      <max_wheel_acceleration>1.8</max_wheel_acceleration>
-      <odom_publish_frequency>1</odom_publish_frequency>
+        <left_joint>left_wheel_joint</left_joint>
+        <right_joint>right_wheel_joint</right_joint>
+        <wheel_separation>${2*base_radius}</wheel_separation>
+        <wheel_radius>${wheel_radius}</wheel_radius>
+        <odom_publish_frequency>10</odom_publish_frequency>
+        <topic>cmd_vel</topic>
+        <!--<robotBaseFrame>base_footprint</robotBaseFrame>-->
+        <ignition_frame_id>base_footprint</ignition_frame_id>
       <!--<ros>
         <namespace>/fra2mo</namespace>

File: urdf/lidar_gazebo_macro.xacro (robot description, xacro)
@@ -22,26 +22,4 @@
         </geometry>
       </collision>
-      <gazebo>
-      <sensor type="gpu_lidar" name="gpu_lidar">
-        <update_rate>40</update_rate>
-        <ray>
-          <scan>
-            <horizontal>
-              <samples>720</samples>
-              <resolution>1</resolution>
-              <min_angle>-3.14</min_angle>
-              <max_angle>3.14</max_angle>
-            </horizontal>
-          </scan>
-          <range>
-            <min>0.1</min>
-            <max>10.0</max>
-            <resolution>0.01</resolution>
-          </range>
-        </ray>
-        <always_on>1</always_on>
-        <visualize>true</visualize>
-      </sensor>
-      </gazebo>
     </link>
     <joint name="laser_joint" type="fixed">
@@ -50,4 +28,41 @@
       <origin rpy="0 0 0" xyz="0.0 0.0 0.031" />
     </joint>
+    <gazebo reference="laser_frame">
+      <sensor name="laser_frame" type="gpu_lidar">
+          <pose relative_to="laser_frame">0 0 0 0 0 0</pose>
+          <topic>lidar</topic>
+          <update_rate>10</update_rate>
+          <ray>
+              <scan>
+                  <horizontal>
+                      <samples>640</samples>
+                      <resolution>1</resolution>
+                      <min_angle>-3.14</min_angle>
+                      <max_angle>3.14</max_angle>
+                  </horizontal>
+                  <!--<vertical>
+                      <samples>1</samples>
+                      <resolution>1</resolution>
+                      <min_angle>-0.261799</min_angle>
+                      <max_angle>0.261799</max_angle>
+                  </vertical>-->
+              </scan>
+              <range>
+                  <min>0.1</min>
+                  <max>10.0</max>
+                  <resolution>0.01</resolution>
+              </range>
+          </ray>
+          <always_on>1</always_on>
+          <visualize>true</visualize>
+         <ignition_frame_id>fra2mo::base_footprint::laser_frame</ignition_frame_id>
+      </sensor>
+  </gazebo>
+  <gazebo>
+    <plugin filename="libignition-gazebo-sensors-system.so"
+      name="ignition::gazebo::systems::Sensors">
+        <render_engine>ogre2</render_engine>
+    </plugin>
+  </gazebo>
   </xacro:macro>
 </robot>
